Commit message: update

File: install/poc_arm/share/poc_arm/urdf/camera_rgbd.xacro (robot description, xacro)
@@ -47,5 +47,5 @@
           </image>
           <clip>
-            <near>0.1</near>
+            <near>0.01</near>
             <far>10.0</far>
           </clip>

File: install/poc_arm/share/poc_arm/urdf/poc_arm_sim.urdf.xacro (robot description, xacro)
@@ -27,5 +27,5 @@
       <geometry>
         <!-- size = X Y Z -->
-        <box size="0.1 0.15 0.50"/>
+        <box size="0.06 0.10 0.50"/>
       </geometry>
       <material name="torso_color">
@@ -36,5 +36,5 @@
       <origin xyz="0 0 0.25" rpy="0 0 0"/>
       <geometry>
-        <box size="0.1 0.15 0.50"/>
+        <box size="0.06 0.10 0.50"/>
       </geometry>
     </collision>
@@ -42,5 +42,5 @@
   <xacro:rgbd_camera
     parent="torso_link"
-    xyz="0.075 0 0.47"
+    xyz="0.065 0 0.47"
     rpy="0 0.4 0"/>
   <link
@@ -66,5 +66,5 @@
       <geometry>
         <mesh
-          filename="${poc_arm_pkg}/meshes/shoulder_base_link.STL" />
+          filename="file:///home/suvi/poc_arm/install/poc_arm/share/poc_arm/meshes/shoulder_base_link.STL" />
       </geometry>
       <material name="grey"/>
@@ -76,5 +76,5 @@
       <geometry>
         <mesh
-          filename="${poc_arm_pkg}/meshes/shoulder_base_link.STL" />
+          filename="file:///home/suvi/poc_arm/install/poc_arm/share/poc_arm/meshes/shoulder_base_link.STL" />
       </geometry>
     </collision>
@@ -85,5 +85,5 @@
     <child link="shoulder_base_link"/>
     <!-- adjust this offset to place your arm on top of torso -->
-    <origin xyz="0 -0.06 0.45" rpy="0 0 0"/>
+    <origin xyz="0 -0.06 0.4" rpy="0 0 0"/>
   </joint>
   <link
@@ -109,5 +109,5 @@
       <geometry>
         <mesh
-          filename="${poc_arm_pkg}/meshes/shoulder_pitch_link.STL" />
+          filename="file:///home/suvi/poc_arm/install/poc_arm/share/poc_arm/meshes/shoulder_pitch_link.STL" />
       </geometry>
       <material name="blue"/>
@@ -119,5 +119,5 @@
       <geometry>
         <mesh
-          filename="${poc_arm_pkg}/meshes/shoulder_pitch_link.STL" />
+          filename="file:///home/suvi/poc_arm/install/poc_arm/share/poc_arm/meshes/shoulder_pitch_link.STL" />
       </geometry>
     </collision>
@@ -163,5 +163,5 @@
       <geometry>
         <mesh
-          filename="${poc_arm_pkg}/meshes/shoulder_yaw_link.STL" />
+          filename="file:///home/suvi/poc_arm/install/poc_arm/share/poc_arm/meshes/shoulder_yaw_link.STL" />
       </geometry>
       <material name="green"/>
@@ -173,5 +173,5 @@
       <geometry>
         <mesh
-          filename="${poc_arm_pkg}/meshes/shoulder_yaw_link.STL" />
+          filename="file:///home/suvi/poc_arm/install/poc_arm/share/poc_arm/meshes/shoulder_yaw_link.STL" />
       </geometry>
     </collision>
@@ -217,5 +217,5 @@
       <geometry>
         <mesh
-          filename="${poc_arm_pkg}/meshes/shoulder_roll_link.STL" />
+          filename="file:///home/suvi/poc_arm/install/poc_arm/share/poc_arm/meshes/shoulder_roll_link.STL" />
       </geometry>
       <material name="grey"/>
@@ -227,5 +227,5 @@
       <geometry>
         <mesh
-          filename="${poc_arm_pkg}/meshes/shoulder_roll_link.STL" />
+          filename="file:///home/suvi/poc_arm/install/poc_arm/share/poc_arm/meshes/shoulder_roll_link.STL" />
       </geometry>
     </collision>
@@ -271,5 +271,5 @@
       <geometry>
         <mesh
-          filename="${poc_arm_pkg}/meshes/elbow_link.STL" />
+          filename="file:///home/suvi/poc_arm/install/poc_arm/share/poc_arm/meshes/elbow_link.STL" />
       </geometry>
       <material name="blue"/>
@@ -281,5 +281,5 @@
       <geometry>
         <mesh
-          filename="${poc_arm_pkg}/meshes/elbow_link.STL" />
+          filename="file:///home/suvi/poc_arm/install/poc_arm/share/poc_arm/meshes/elbow_link.STL" />
       </geometry>
     </collision>
@@ -325,5 +325,5 @@
       <geometry>
         <mesh
-          filename="${poc_arm_pkg}/meshes/wrist_yaw_link.STL" />
+          filename="file:///home/suvi/poc_arm/install/poc_arm/share/poc_arm/meshes/wrist_yaw_link.STL" />
       </geometry>
       <material name="green"/>
@@ -335,5 +335,5 @@
       <geometry>
         <mesh
-          filename="${poc_arm_pkg}/meshes/wrist_yaw_link.STL" />
+          filename="file:///home/suvi/poc_arm/install/poc_arm/share/poc_arm/meshes/wrist_yaw_link.STL" />
       </geometry>
     </collision>
@@ -379,5 +379,5 @@
       <geometry>
         <mesh
-          filename="${poc_arm_pkg}/meshes/wrist_pitch_link.STL" />
+          filename="file:///home/suvi/poc_arm/install/poc_arm/share/poc_arm/meshes/wrist_pitch_link.STL" />
       </geometry>
       <material name="grey"/>
@@ -389,5 +389,5 @@
       <geometry>
         <mesh
-          filename="${poc_arm_pkg}/meshes/wrist_pitch_link.STL" />
+          filename="file:///home/suvi/poc_arm/install/poc_arm/share/poc_arm/meshes/wrist_pitch_link.STL" />
       </geometry>
     </collision>
@@ -433,5 +433,5 @@
       <geometry>
         <mesh
-          filename="${poc_arm_pkg}/meshes/wrist_roll_link.STL" />
+          filename="file:///home/suvi/poc_arm/install/poc_arm/share/poc_arm/meshes/wrist_roll_link.STL" />
       </geometry>
       <material name="blue"/>
@@ -443,5 +443,5 @@
       <geometry>
         <mesh
-          filename="${poc_arm_pkg}/meshes/wrist_roll_link.STL" />
+          filename="file:///home/suvi/poc_arm/install/poc_arm/share/poc_arm/meshes/wrist_roll_link.STL" />
       </geometry>
     </collision>

Commit message: update

File: install/poc_arm/share/poc_arm/urdf/camera_rgbd.xacro (robot description, xacro)
@@ -2,8 +2,13 @@
 <robot xmlns:xacro="http://www.ros.org/wiki/xacro">
   <xacro:macro name="rgbd_camera" params="parent xyz rpy">
-  <material name="black">
-      <color rgba="0 0 0 1" />
-  </material>
-    <!-- Camera link -->
+    <!-- ================= -->
+    <!-- Materials -->
+    <!-- ================= -->
+    <material name="black">
+      <color rgba="0 0 0 1"/>
+    </material>
+    <!-- ================= -->
+    <!-- Camera mounting link -->
+    <!-- ================= -->
     <link name="camera_link">
       <inertial>
@@ -28,39 +33,52 @@
       </collision>
     </link>
-    <!-- Fixed joint to parent -->
-    <joint name="camera_fixed_joint" type="fixed">
+    <!-- ================= -->
+    <!-- Optical frame link -->
+    <!-- ================= -->
+    <link name="camera_frame_link"/>
+    <!-- ================= -->
+    <!-- Parent → camera_link -->
+    <!-- ================= -->
+    <joint name="head_to_camera_link" type="fixed">
       <parent link="${parent}"/>
       <child link="camera_link"/>
       <origin xyz="${xyz}" rpy="${rpy}"/>
     </joint>
+    <!-- ================= -->
+    <!-- camera_link → camera_frame_link (REP-103 optical frame) -->
+    <!-- ================= -->
+    <joint name="camera_link_to_camera_frame_link" type="fixed">
+      <parent link="camera_link"/>
+      <child link="camera_frame_link"/>
+      <origin xyz="0 0 0" rpy="-1.57 0 -1.57"/>
+    </joint>
+    <!-- ================= -->
     <!-- Gazebo RGB-D sensor -->
-    <gazebo reference="camera_link">
-      <sensor type="depth" name="rgbd_camera">
-        <always_on>true</always_on>
-        <update_rate>30</update_rate>
-        <camera>
-          <horizontal_fov>1.57</horizontal_fov>
-          <image>
-            <width>640</width>
-            <height>480</height>
-            <format>R8G8B8</format>
-          </image>
-          <clip>
-            <near>0.01</near>
-            <far>10.0</far>
-          </clip>
-        </camera>
-        <plugin name="rgbd_camera_controller" filename="libgazebo_ros_camera.so">
-          <camera_name>camera</camera_name>
-          <frame_name>camera_link</frame_name>
-          <image_topic_name>color/image_raw</image_topic_name>
-          <camera_info_topic_name>color/camera_info</camera_info_topic_name>
-          <depth_image_topic_name>depth/image_raw</depth_image_topic_name>
-          <depth_camera_info_topic_name>depth/camera_info</depth_camera_info_topic_name>
-          <point_cloud>true</point_cloud>
-          <point_cloud_topic_name>depth/points</point_cloud_topic_name>
-        </plugin>
-      </sensor>
-    </gazebo>
+    <!-- ================= -->
+    <xacro:if value="true">
+      <gazebo reference="camera_link">
+        <sensor name="camera" type="depth">
+          <pose>0 0 0 0 0 0</pose>
+          <visualize>true</visualize>
+          <update_rate>5</update_rate>
+          <camera>
+            <horizontal_fov>2</horizontal_fov>
+            <image>
+              <format>R8G8B8</format>
+              <width>640</width>
+              <height>480</height>
+            </image>
+            <clip>
+              <near>0.2</near>
+              <far>5</far>
+            </clip>
+          </camera>
+          <plugin name="depth_camera" filename="libgazebo_ros_camera.so">
+            <!-- Optical frame -->
+            <frame_name>camera_frame_link</frame_name>
+          </plugin>
+        </sensor>
+      </gazebo>
+    </xacro:if>
   </xacro:macro>
 </robot>

File: install/poc_arm/share/poc_arm/urdf/poc_arm_sim.urdf.xacro (robot description, xacro)
@@ -17,5 +17,5 @@
     <inertial>
       <origin xyz="0 0 0.25" rpy="0 0 0"/>
-      <mass value="25"/>
+      <mass value="250"/>
       <inertia
         ixx="0.2" ixy="0.0" ixz="0.0"
@@ -42,6 +42,6 @@
   <xacro:rgbd_camera
     parent="torso_link"
-    xyz="0.065 0 0.35"
-    rpy="0 0 0"/>
+    xyz="0.015 0 0.75"
+    rpy="0 0.45 0"/>
   <link
     name="shoulder_base_link">

File: src/poc_arm/urdf/poc_arm_sim.urdf.xacro (robot description, xacro)
@@ -17,5 +17,5 @@
     <inertial>
       <origin xyz="0 0 0.25" rpy="0 0 0"/>
-      <mass value="25"/>
+      <mass value="250"/>
       <inertia
         ixx="0.2" ixy="0.0" ixz="0.0"
@@ -42,6 +42,6 @@
   <xacro:rgbd_camera
     parent="torso_link"
-    xyz="0.065 0 0.47"
-    rpy="0 0.4 0"/>
+    xyz="0.015 0 0.75"
+    rpy="0 0.45 0"/>
   <link
     name="shoulder_base_link">
