Commit message: update

File: install/poc_arm/share/poc_arm/urdf/poc_arm_sim.urdf.xacro (robot description, xacro)
@@ -2,4 +2,5 @@
 <robot name="my_robot"
        xmlns:xacro="http://www.ros.org/wiki/xacro">
+  <xacro:include filename="$(find poc_arm)/urdf/camera_rgbd.xacro"/>
   <material name="grey">
       <color rgba="0.5 0.5 0.5 1" />
@@ -16,5 +17,5 @@
     <inertial>
       <origin xyz="0 0 0.25" rpy="0 0 0"/>
-      <mass value="20"/>
+      <mass value="25"/>
       <inertia
         ixx="0.2" ixy="0.0" ixz="0.0"
@@ -26,5 +27,5 @@
       <geometry>
         <!-- size = X Y Z -->
-        <box size="0.06 0.10 0.50"/>
+        <box size="0.1 0.15 0.50"/>
       </geometry>
       <material name="torso_color">
@@ -35,8 +36,12 @@
       <origin xyz="0 0 0.25" rpy="0 0 0"/>
       <geometry>
-        <box size="0.06 0.10 0.50"/>
-      </geometry>
-    </collision>
-  </link>
+        <box size="0.1 0.15 0.50"/>
+      </geometry>
+    </collision>
+  </link>
+  <xacro:rgbd_camera
+    parent="torso_link"
+    xyz="0.075 0 0.47"
+    rpy="0 0.4 0"/>
   <link
     name="shoulder_base_link">
@@ -80,5 +85,5 @@
     <child link="shoulder_base_link"/>
     <!-- adjust this offset to place your arm on top of torso -->
-    <origin xyz="0 -0.06 0.40" rpy="0 0 0"/>
+    <origin xyz="0 -0.06 0.45" rpy="0 0 0"/>
   </joint>
   <link
@@ -463,4 +468,7 @@
       <material>Gazebo/White</material>
   </gazebo>
+  <gazebo reference="camera_link">
+      <material>Gazebo/Black</material>
+  </gazebo>
   <gazebo reference="shoulder_base_link">
       <material>Gazebo/Grey</material>

File: src/realsense_gazebo/urdf/camera_bot_rs.urdf (robot description, URDF)
Before this commit: robot camera_bot, 2 links, 1 joints
Links:
- removed link base_link
Joints:
- removed joint camera_joint

Commit message: update

File: install/poc_arm/share/poc_arm/urdf/poc_arm_sim.urdf.xacro (robot description, xacro)
@@ -85,5 +85,5 @@
     <child link="shoulder_base_link"/>
     <!-- adjust this offset to place your arm on top of torso -->
-    <origin xyz="0 -0.06 0.4" rpy="0 0 0"/>
+    <origin xyz="0 -0.06 0.45" rpy="0 0 0"/>
   </joint>
   <link

Commit message: update

File: install/poc_arm/share/poc_arm/urdf/poc_arm_sim.urdf.xacro (robot description, xacro)
@@ -85,5 +85,5 @@
     <child link="shoulder_base_link"/>
     <!-- adjust this offset to place your arm on top of torso -->
-    <origin xyz="0 -0.06 0.45" rpy="0 0 0"/>
+    <origin xyz="0 -0.06 0.4" rpy="0 0 0"/>
   </joint>
   <link
