Commit message: update

File: src/poc_arm/urdf/poc_arm_real.urdf.xacro (robot description, xacro)
@@ -12,5 +12,4 @@
       <color rgba="0 0.4 0 1" />
   </material>
-  <xacro:property name="poc_arm_pkg" value="$(find poc_arm)"/>
   <!-- Torso / base box -->
   <link name="torso_link">
@@ -66,5 +65,5 @@
       <geometry>
         <mesh
-          filename="file:///home/suvi/poc_arm/install/poc_arm/share/poc_arm/meshes/shoulder_base_link.STL" />
+          filename="package://poc_arm/meshes/shoulder_base_link.STL" />
       </geometry>
       <material name="grey"/>
@@ -76,5 +75,5 @@
       <geometry>
         <mesh
-          filename="file:///home/suvi/poc_arm/install/poc_arm/share/poc_arm/meshes/shoulder_base_link.STL" />
+          filename="package://poc_arm/meshes/shoulder_base_link.STL" />
       </geometry>
     </collision>
@@ -109,5 +108,5 @@
       <geometry>
         <mesh
-          filename="file:///home/suvi/poc_arm/install/poc_arm/share/poc_arm/meshes/shoulder_pitch_link.STL" />
+          filename="package://poc_arm/meshes/shoulder_pitch_link.STL" />
       </geometry>
       <material name="blue"/>
@@ -119,5 +118,5 @@
       <geometry>
         <mesh
-          filename="file:///home/suvi/poc_arm/install/poc_arm/share/poc_arm/meshes/shoulder_pitch_link.STL" />
+          filename="package://poc_arm/meshes/shoulder_pitch_link.STL" />
       </geometry>
     </collision>
@@ -163,5 +162,5 @@
       <geometry>
         <mesh
-          filename="file:///home/suvi/poc_arm/install/poc_arm/share/poc_arm/meshes/shoulder_yaw_link.STL" />
+          filename="package://poc_arm/meshes/shoulder_yaw_link.STL" />
       </geometry>
       <material name="green"/>
@@ -173,5 +172,5 @@
       <geometry>
         <mesh
-          filename="file:///home/suvi/poc_arm/install/poc_arm/share/poc_arm/meshes/shoulder_yaw_link.STL" />
+          filename="package://poc_arm/meshes/shoulder_yaw_link.STL" />
       </geometry>
     </collision>
@@ -217,5 +216,5 @@
       <geometry>
         <mesh
-          filename="file:///home/suvi/poc_arm/install/poc_arm/share/poc_arm/meshes/shoulder_roll_link.STL" />
+          filename="package://poc_arm/meshes/shoulder_roll_link.STL" />
       </geometry>
       <material name="grey"/>
@@ -227,5 +226,5 @@
       <geometry>
         <mesh
-          filename="file:///home/suvi/poc_arm/install/poc_arm/share/poc_arm/meshes/shoulder_roll_link.STL" />
+          filename="package://poc_arm/meshes/shoulder_roll_link.STL" />
       </geometry>
     </collision>
@@ -271,5 +270,5 @@
       <geometry>
         <mesh
-          filename="file:///home/suvi/poc_arm/install/poc_arm/share/poc_arm/meshes/elbow_link.STL" />
+          filename="package://poc_arm/meshes/elbow_link.STL" />
       </geometry>
       <material name="blue"/>
@@ -281,5 +280,5 @@
       <geometry>
         <mesh
-          filename="file:///home/suvi/poc_arm/install/poc_arm/share/poc_arm/meshes/elbow_link.STL" />
+          filename="package://poc_arm/meshes/elbow_link.STL" />
       </geometry>
     </collision>
@@ -325,5 +324,5 @@
       <geometry>
         <mesh
-          filename="file:///home/suvi/poc_arm/install/poc_arm/share/poc_arm/meshes/wrist_yaw_link.STL" />
+          filename="package://poc_arm/meshes/wrist_yaw_link.STL" />
       </geometry>
       <material name="green"/>
@@ -335,5 +334,5 @@
       <geometry>
         <mesh
-          filename="file:///home/suvi/poc_arm/install/poc_arm/share/poc_arm/meshes/wrist_yaw_link.STL" />
+          filename="package://poc_arm/meshes/wrist_yaw_link.STL" />
       </geometry>
     </collision>
@@ -379,5 +378,5 @@
       <geometry>
         <mesh
-          filename="file:///home/suvi/poc_arm/install/poc_arm/share/poc_arm/meshes/wrist_pitch_link.STL" />
+          filename="package://poc_arm/meshes/wrist_pitch_link.STL" />
       </geometry>
       <material name="grey"/>
@@ -389,5 +388,5 @@
       <geometry>
         <mesh
-          filename="file:///home/suvi/poc_arm/install/poc_arm/share/poc_arm/meshes/wrist_pitch_link.STL" />
+          filename="package://poc_arm/meshes/wrist_pitch_link.STL" />
       </geometry>
     </collision>
@@ -433,5 +432,5 @@
       <geometry>
         <mesh
-          filename="file:///home/suvi/poc_arm/install/poc_arm/share/poc_arm/meshes/wrist_roll_link.STL" />
+          filename="package://poc_arm/meshes/wrist_roll_link.STL" />
       </geometry>
       <material name="blue"/>
@@ -443,5 +442,5 @@
       <geometry>
         <mesh
-          filename="file:///home/suvi/poc_arm/install/poc_arm/share/poc_arm/meshes/wrist_roll_link.STL" />
+          filename="package://poc_arm/meshes/wrist_roll_link.STL" />
       </geometry>
     </collision>
